File: KiCad/Clever_Light.sch (KiCad schematic (older format))
At the start: 14 parts, among them IC1 BTA08-600SWRG, J1 Screw_Terminal_01x02, J2 Screw_Terminal_01x02, J3 Screw_Terminal_01x02, J4 Screw_Terminal_01x02, J5 Conn_02x07_Odd_Even, Q1 SFH6156-3T, U1 MOC3063M

Commit message: правка пинов
Parts:
- IC1: symbol BTA08-600SWRG:BTA08-600SWRG -> Clever_Light-rescue:BTA08-600SWRG-BTA08-600SWRG
- Q1: symbol SFH6156-3T:SFH6156-3T -> Clever_Light-rescue:SFH6156-3T-SFH6156-3T
Changed lines of the file:
@@
 $EndComp
 $Comp
-L BTA08-600SWRG:BTA08-600SWRG IC1
+L Clever_Light-rescue:BTA08-600SWRG-BTA08-600SWRG IC1
 U 1 1 5D3A683B
 P 3650 2150
@@
 NoConn ~ 4650 2400
 $Comp
-L SFH6156-3T:SFH6156-3T Q1
+L Clever_Light-rescue:SFH6156-3T-SFH6156-3T Q1
 U 1 1 5D3C0E10
 P 1650 1100

Commit message: небольшая оптимизация
Parts:
- IC1: footprint Package_TO_SOT_THT:TO-220-3_Horizontal_TabUp -> Package_TO_SOT_THT:TO-220-3_Horizontal_TabDown
- J1, J2, J3, J4: footprint TerminalBlock_Phoenix:TerminalBlock_Phoenix_PT-1,5-2-5.0-H_1x02_P5.00mm_Horizontal -> TerminalBlock_Phoenix:TerminalBlock_KV301_1x02_P5.00mm_Horizontal
- R1, R3: footprint Resistor_THT:R_Axial_DIN0204_L3.6mm_D1.6mm_P7.62mm_Horizontal -> Resistor_SMD:R_1206_3216Metric
- R2, R6: footprint Resistor_SMD:R_1206_3216Metric_Pad1.42x1.75mm_HandSolder -> Resistor_SMD:R_1206_3216Metric
Changed lines of the file:
@@
 EESchema Schematic File Version 4
 LIBS:Clever_Light-cache
-EELAYER 29 0
+EELAYER 30 0
 EELAYER END
 $Descr A4 11693 8268
@@
 F 0 "R3" V 1600 1950 50  0000 C CNN
 F 1 "680" V 1500 1950 50  0000 C CNN
-F 2 "Resistor_THT:R_Axial_DIN0204_L3.6mm_D1.6mm_P7.62mm_Horizontal" V 1430 1950 50  0001 C CNN
+F 2 "Resistor_SMD:R_1206_3216Metric" V 1430 1950 50  0001 C CNN
 F 3 "~" H 1500 1950 50  0001 C CNN
 	1    1500 1950
@@
 F 0 "R1" V 1400 1000 50  0000 C CNN
 F 1 "2.2k" V 1300 1000 50  0000 C CNN
-F 2 "Resistor_THT:R_Axial_DIN0204_L3.6mm_D1.6mm_P7.62mm_Horizontal" V 1230 1000 50  0001 C CNN
+F 2 "Resistor_SMD:R_1206_3216Metric" V 1230 1000 50  0001 C CNN
 F 3 "~" H 1300 1000 50  0001 C CNN
 	1    1300 1000
@@
 F 0 "R2" V 2900 1000 50  0000 C CNN
 F 1 "4.7k" V 3000 1000 50  0000 C CNN
-F 2 "Resistor_SMD:R_1206_3216Metric_Pad1.42x1.75mm_HandSolder" V 2930 1000 50  0001 C CNN
+F 2 "Resistor_SMD:R_1206_3216Metric" V 2930 1000 50  0001 C CNN
 F 3 "~" H 3000 1000 50  0001 C CNN
 	1    3000 1000
@@
 F 0 "IC1" H 4100 1900 50  0000 C CNN
 F 1 "BTA08-600SWRG" H 4100 2300 50  0000 C CNN
-F 2 "Package_TO_SOT_THT:TO-220-3_Horizontal_TabUp" H 4400 2250 50  0001 L CNN
+F 2 "Package_TO_SOT_THT:TO-220-3_Horizontal_TabDown" H 4400 2250 50  0001 L CNN
 F 3 "https://componentsearchengine.com/Datasheets/1/BTA08-600SWRG.pdf" H 4400 2150 50  0001 L CNN
 F 4 "" H 4400 2050 50  0001 L CNN "Description"
@@
 F 0 "J4" V 7800 1000 50  0000 C CNN
 F 1 "Screw_Terminal_01x02" V 7700 1000 50  0000 C CNN
-F 2 "TerminalBlock_Phoenix:TerminalBlock_Phoenix_PT-1,5-2-5.0-H_1x02_P5.00mm_Horizontal" H 7550 1050 50  0001 C CNN
+F 2 "TerminalBlock_Phoenix:TerminalBlock_KV301_1x02_P5.00mm_Horizontal" H 7550 1050 50  0001 C CNN
 F 3 "~" H 7550 1050 50  0001 C CNN
 	1    7550 1050
@@
 F 0 "J3" V 6850 1000 50  0000 C CNN
 F 1 "Screw_Terminal_01x02" V 6750 1000 50  0000 C CNN
-F 2 "TerminalBlock_Phoenix:TerminalBlock_Phoenix_PT-1,5-2-5.0-H_1x02_P5.00mm_Horizontal" H 6600 1050 50  0001 C CNN
+F 2 "TerminalBlock_Phoenix:TerminalBlock_KV301_1x02_P5.00mm_Horizontal" H 6600 1050 50  0001 C CNN
 F 3 "~" H 6600 1050 50  0001 C CNN
 	1    6600 1050
@@
 F 0 "J2" V 5900 1000 50  0000 C CNN
 F 1 "Screw_Terminal_01x02" V 5800 1000 50  0000 C CNN
-F 2 "TerminalBlock_Phoenix:TerminalBlock_Phoenix_PT-1,5-2-5.0-H_1x02_P5.00mm_Horizontal" H 5650 1050 50  0001 C CNN
+F 2 "TerminalBlock_Phoenix:TerminalBlock_KV301_1x02_P5.00mm_Horizontal" H 5650 1050 50  0001 C CNN
 F 3 "~" H 5650 1050 50  0001 C CNN
 	1    5650 1050
@@
 F 0 "J1" V 4950 1000 50  0000 C CNN
 F 1 "Screw_Terminal_01x02" V 4850 1000 50  0000 C CNN
-F 2 "TerminalBlock_Phoenix:TerminalBlock_Phoenix_PT-1,5-2-5.0-H_1x02_P5.00mm_Horizontal" H 4700 1050 50  0001 C CNN
+F 2 "TerminalBlock_Phoenix:TerminalBlock_KV301_1x02_P5.00mm_Horizontal" H 4700 1050 50  0001 C CNN
 F 3 "~" H 4700 1050 50  0001 C CNN
 	1    4700 1050
@@
 F 0 "R6" H 5650 2150 50  0000 C CNN
 F 1 "4.7k" V 5750 2150 50  0000 C CNN
-F 2 "Resistor_SMD:R_1206_3216Metric_Pad1.42x1.75mm_HandSolder" V 5680 2150 50  0001 C CNN
+F 2 "Resistor_SMD:R_1206_3216Metric" V 5680 2150 50  0001 C CNN
 F 3 "~" H 5750 2150 50  0001 C CNN
 	1    5750 2150
